Commit message: Indent URDF in a tree structure

File: src/darwin_description/urdf/mydarwin.urdf (robot description, URDF)
Before this commit: robot darwinOP, 31 links, 30 joints
Links:
- removed link ARM_GRIPPER_FIX_DUMMY_L
- removed link ARM_GRIPPER_FIX_DUMMY_R
- removed link PMDCAMBOARD
Joints:
- removed joint j_camboard
- removed joint j_wrist_dummy_l
- removed joint j_wrist_dummy_r
- joint j_gripper_l: axis 0 0 1 -> (none); limit lower=-2.6179939 upper=2.6179939 effort=2.8 velocity=5.6548668 -> (none); origin xyz=0.048 0.01 0 rpy=0 0 1.0 -> xyz=0.048 0.01 0 rpy=0 0 0; type revolute -> fixed
- joint j_gripper_r: axis 0 0 1 -> (none); limit lower=-2.6179939 upper=2.6179939 effort=2.8 velocity=5.6548668 -> (none); origin xyz=0.048 0.01 0 rpy=0 0 1.0 -> xyz=0.048 0.01 0 rpy=0 0 0; type revolute -> fixed
- joint j_wrist_l: axis 0 0 1 -> (none); limit lower=-2.6179939 upper=2.6179939 effort=2.8 velocity=5.6548668 -> (none); type revolute -> fixed
- joint j_wrist_r: axis 0 0 1 -> (none); limit lower=-2.6179939 upper=2.6179939 effort=2.8 velocity=5.6548668 -> (none); type revolute -> fixed
